File: MH-M38 Eagle circuit.sch (EAGLE design)
At the start: 28 parts, among them J1 CON-2P, J2 CON-3P, J3 CON-2P, U1 MH-M38, U2 TC8871, U3 TC8871, Y1 24MHz, Y2 XRCGB24M000F3N00R0

Commit message: Add files via upload
Parts:
- removed Y2: XRCGB24M000F3N00R0, Albert:CRYSTAL-SMD128
- added C14: 1u 6.3V, Albert:SMD-C-0402-SMALL
- added J4: USB-MICRO-B", Albert:USB-MICRO-B"
- added R5: 10k, Albert:SMD-R-0402-SMALL
- C1: value 10u 6.3V -> 8u 0402
- C12: value 1u 6.3V -> 10u 6.3V 0603; device Albert:SMD-C-0402-SMALL -> Albert:SMD-C-0603-SMALL
- R2: value 10k -> 0E
Connections:
- removed net N$5: D2.A, J2.2
- new net N$22: J4.D+, U1.USB-D+
- new net N$27: C5.2, C6.2, R2.1, U1.GND2
- new net N$28: J4.D-, U1.USB-D-
- new net N$29: D2.A, J2.2, J4.VBUS
- net 3.7V1: now also C13.1, R5.2; no longer R4.2
- net GND: now also C14.2, J4.GND, R2.2; no longer C5.2, C6.2, U1.GND2
- net N$14: now also R3.1; no longer R2.1
- net N$16: now also R4.1; no longer R3.1
- net N$17: now also R3.2; no longer R2.2
- net N$20: now also R5.1, U1.X; no longer R4.1, U1.MUTE-OUT?
- net N$21: now also C14.1; no longer C13.1
- net N$25: now also R4.2; no longer R3.2
Other:
- note added: "Should mute U2/U3 but it is always 0V"
- note added: "Why R5?"
- moved on the sheet: C12, C13, C8, J2, J3, R2, R3, R4
